File: circuts/jut-sweep/digits.sch (KiCad schematic (older format))
At the start: 192 parts, among them IC1 ATMEGA88PA-A, K1 momis, P1 CONN_1, P2 uart, P3 CONN_2, P4 CONN_2, P5 CONN_2, Q1 MOSFET_N, Q10 MOSFET_N, Q11 MOSFET_N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

Commit message: First schematic, made by masa
Connections:
- net at Q3.G: now also IC1.27 ((PCINT12/SDA/ADC4)PC4); no longer IC1.13 ((PCINT1/OC1A)PB1)
- net at Q6.G: now also IC1.26 ((PCINT11/ADC3)PC3); no longer IC1.14 ((PCINT2/OC1B/~SS~)PB2)
- net at IC1.16 ((PCINT4/MISO)PB4), K1.2 (PM): now also Q8.G; no longer Q7.G
- net at Q4.G: now also IC1.17 ((PCINT5/SCK)PB5), K1.1 (P1); no longer IC1.11 ((PCINT23/AIN1)PD7)
- net at IC1.24 ((PCINT9/ADC1)PC1): now also Q7.G; no longer Q9.G
- net at Q11.G: now also IC1.13 ((PCINT1/OC1A)PB1); no longer IC1.26 ((PCINT11/ADC3)PC3)
- net at IC1.25 ((PCINT10/ADC2)PC2): now also Q1.G; no longer Q10.G
- net at Q12.G: now also IC1.12 ((PCINT0/CLKO/ICP1)PB0); no longer IC1.27 ((PCINT12/SDA/ADC4)PC4)
- net at Q13.G: now also IC1.11 ((PCINT23/AIN1)PD7); no longer IC1.28 ((PCINT14/SCL/ADC5)PC5)
- net at IC1.23 ((PCINT8/ADC0)PC0): now also Q2.G; no longer Q8.G
- net at Q5.G: now also IC1.28 ((PCINT14/SCL/ADC5)PC5); no longer IC1.12 ((PCINT0/CLKO/ICP1)PB0)
- new net: IC1.15 ((PCINT3/OC2A/MOSI)PB3), K1.3 (P3), Q9.G
- new net: IC1.14 ((PCINT2/OC1B/~SS~)PB2), Q10.G
